Commit message: four wheek robot wheel macro

File: urdf/robot.xacro (robot description, xacro)
@@ -62,13 +62,31 @@
       <visual>
         <!-- TODO: Complete -->
+        <geometry>
+          <cylinder radius="${wheel_link_radius}" length="${wheel_link_length}"/>
+        </geometry>
+        <origin rpy="1.5708 0 0" xyz="0 0 0"/>
       </visual>
       <collision>
         <!-- TODO: Complete -->
+        <geometry>
+          <cylinder radius="${wheel_link_radius}" length="${wheel_link_length}"/>
+        </geometry>
+        <origin rpy="1.5708 0 0" xyz="0 0 0"/>
       </collision>
       <inertial>
         <!-- TODO: Complete -->
+        <origin xyz="0 0 0" rpy="0 0 0"/> <!--pose of the inertial frame relative to the link's reference frame-->
+        <mass value="${wheel_mass}"/>
+        <inertia
+          ixx="I_wheel" iyy="I_wheel" izz="${Iz_wheel}"
+          ixy="0.0" ixz="0.0" iyz="0.0"
+        />
     </link>
     <joint name="${name}_joint" type="${joint_type}">
       <!-- TODO: Complete -->
+      <parent link="body_link"/>
+      <child link="${name}"/>
+      <origin xyz="${x} ${y} ${z}"/>
+      <axis xyz="0 0 1"/>
       <limit effort="1000" velocity="1000"/>
       <dynamics damping="1.0" friction="1.0"/>
@@ -78,4 +96,7 @@
   <xacro:wheel name="rear_right_wheel"  x="${-body_link_x_dim/2 + 1.2*wheel_link_radius}" y="${-body_link_y_dim/2 - 1.2*wheel_link_length/2}" z="${wheel_link_z_location}" joint_type="continuous"/>
   <!-- TODO: Complete: Wheels must be named - rear_left_wheel, front_right_wheel, front_left_wheel -->
+  <xacro:wheel name="rear_left_wheel"   x="${-body_link_x_dim/2 + 1.2*wheel_link_radius}" y="${ body_link_y_dim/2 + 1.2*wheel_link_length/2}" z="${wheel_link_z_location}" joint_type="continuous"/>
+  <xacro:wheel name="front_right_wheel" x="${ body_link_x_dim/2 - 1.2*wheel_link_radius}" y="${-body_link_y_dim/2 - 1.2*wheel_link_langth/2}" z="${wheel_link_z_location}" joint_type="continuous"/>
+  <xacro:wheel name="front_left_wheel"  x="${ body_link_x_dim/2 - 1.2*wheel_link_radius}" y="${ body_link_y_dim/2 + 1.2*wheel_link_langth/2}" z="${wheel_link_z_location}" joint_type="continuous"/>
 <!-- Camera -->
   <link name="camera_link">

Commit message: xacro file

File: urdf/robot.xacro (robot description, xacro)
@@ -127,11 +127,48 @@
   <link name="sonar_link">
     <!-- TODO: Complete -->
+    <visual>
+      <geometry>
+        <box size="${sensor_side} ${sensor_side} ${sensor_side}"/>
+        <origin rpy="0 0 0" xyz="0 0 0"/>
+      </geometry>
+    </visual>
+    <!--<collision></collision>-->
+    <inertial>
+      <origin rpy="0 0 0" xyz="0 0 0"/>
+      <mass value="${sensor_mass}"/>
+      <inertia
+        ixx="1e-6" ixy="0.0" ixz="0.0"
+        iyy="1e-6" iyz="0.0"
+        izz="1e-6"/> <!--inertia values are small, indicating that sensors are light weight objects, 1e-6 value is used because it is required to have inertia values for objects-->
+    </inertial>
   </link>
   <joint name="sonar_joint" type="fixed">
     <!-- TODO: Complete -->
+    <parent link="body_link"/>
+    <child link="sonar_link"/>
+    <origin xyz="${body_link_x_dim + sensor_side/2} 0 0"/>
+    <axis xyz="0 0 0"/>
   </joint>
   <!-- Lidar -->
   <link name="lidar_link">
     <!-- TODO: Complete -->
+    <visual>
+      <geometry>
+        <box size="${sensor_side} ${sensor_side} ${sensor_side}"/>
+        <origin rpy="0 0 0" xyz="0 0 0"/>
+      </geometry>
+    </visual>
+    <collision>
+      <geometry><box size="${sensor_side} ${sensor_side} ${sensor_side}"/></geometry>
+      <origin rpy="0 0 0" xyz="0 0 0"/>
+    </collision>
+    <inertial>
+      <origin rpy="0 0 0" xyz="0 0 0"/>
+      <mass value="${sensor_mass}"/>
+      <inertia
+        ixx="1e-6" ixy="0.0" ixz="0.0"
+        iyy="1e-6" iyz="0.0"
+        izz="1e-6"/>
+    </inertial>
   </link>
   <joint name="lidar_joint" type="fixed">

Commit message: lidar_joint

File: urdf/robot.xacro (robot description, xacro)
@@ -174,4 +174,7 @@
   <joint name="lidar_joint" type="fixed">
     <!-- TODO: Complete -->
+    <parent link="body_link" />
+    <child link="lidar_link" />
+    <origin xyz="0 0 ${body_link_z_dim/2 + sensor_side/2}"/>
   </joint>
 </robot>

Commit message: solution

File: urdf/robot.xacro (robot description, xacro)
@@ -24,5 +24,5 @@
   <xacro:property name="I_wheel" value="${(1.0/12.0) * wheel_mass * (3.0 * wheel_link_radius * wheel_link_radius + wheel_link_length * wheel_link_length)}"/>
   <!-- Gazebo definitions -->
-  <xacro:include filename="$(find robot_model_pkg)/urdf/robot.gazebo"/>
+  <xacro:include filename="$(find four_wheel_robot)/urdf/robot.gazebo"/>
   <!-- Dummy link -->
   <link name="dummy"/>
@@ -79,7 +79,8 @@
         <mass value="${wheel_mass}"/>
         <inertia
-          ixx="I_wheel" iyy="I_wheel" izz="${Iz_wheel}"
+          ixx="${I_wheel}" iyy="${I_wheel}" izz="${Iz_wheel}"
           ixy="0.0" ixz="0.0" iyz="0.0"
         />
+      </inertial>
     </link>
     <joint name="${name}_joint" type="${joint_type}">
@@ -97,6 +98,6 @@
   <!-- TODO: Complete: Wheels must be named - rear_left_wheel, front_right_wheel, front_left_wheel -->
   <xacro:wheel name="rear_left_wheel"   x="${-body_link_x_dim/2 + 1.2*wheel_link_radius}" y="${ body_link_y_dim/2 + 1.2*wheel_link_length/2}" z="${wheel_link_z_location}" joint_type="continuous"/>
-  <xacro:wheel name="front_right_wheel" x="${ body_link_x_dim/2 - 1.2*wheel_link_radius}" y="${-body_link_y_dim/2 - 1.2*wheel_link_langth/2}" z="${wheel_link_z_location}" joint_type="continuous"/>
-  <xacro:wheel name="front_left_wheel"  x="${ body_link_x_dim/2 - 1.2*wheel_link_radius}" y="${ body_link_y_dim/2 + 1.2*wheel_link_langth/2}" z="${wheel_link_z_location}" joint_type="continuous"/>
+  <xacro:wheel name="front_right_wheel" x="${ body_link_x_dim/2 - 1.2*wheel_link_radius}" y="${-body_link_y_dim/2 - 1.2*wheel_link_length/2}" z="${wheel_link_z_location}" joint_type="continuous"/>
+  <xacro:wheel name="front_left_wheel"  x="${ body_link_x_dim/2 - 1.2*wheel_link_radius}" y="${ body_link_y_dim/2 + 1.2*wheel_link_length/2}" z="${wheel_link_z_location}" joint_type="continuous"/>
 <!-- Camera -->
   <link name="camera_link">
